File: Hardware/STM32G431CBT6-project-template_PROJECT/STM32G431CBT6-project-template.kicad_sch (KiCad schematic)
At the start: 7 parts

Commit message: basic stm32g4 schmatic
Parts:
- removed BT1: Battery, Battery:BatteryHolder_LINX_BAT-HLD-012-SMT, symbol Device:Battery
- removed D1: LED, LED_SMD:LED_0805_2012Metric, symbol Device:LED
- removed R1: R, Resistor_SMD:R_0805_2012Metric, symbol Device:R
Connections:
- no-connect marks 0 -> 22
Other:
- added sheet STM32G4 (stm32g4.kicad_sch)
- added sheet USB-power (usb-power.kicad_sch)
- note removed: "CIRCUIT"
- moved on the sheet: H1, H2, H3, H4
